Commit message: refactor(assets): rename lkls73 → p7 across arm, torso, workstations
Renames the lkls73_arm component to `p7`, lkls73_torso → p7_torso, and the
three lkls73_i1_* workstations to p7_i1_*. Updates all internal identifiers
(URDF robot names, MJCF model + class names, material, recipe/manifest/config
references, docs, and the add_robot_component skill). Recomposes the p7
workstations plus a7_lite dependents so the drift gate is clean.

Refs: #6

File: src/linker_robot_assets/assets/workstations/p7_i1_bimanual/workstation.urdf (robot description, URDF)
Before this commit: robot lkls73_i1_bimanual, 57 links, 56 joints
Links:
- link arm_left_L1_Link: geometry collision mesh filename=../../components/arms/p7/variants/left/meshes/L1_Link.STL; visual mesh filename=../../components/arms/p7/variants/left/meshes/L1_Link.STL
- link arm_left_L2_Link: geometry collision mesh filename=../../components/arms/p7/variants/left/meshes/L2_Link.STL; visual mesh filename=../../components/arms/p7/variants/left/meshes/L2_Link.STL
- link arm_left_L3_Link: geometry collision mesh filename=../../components/arms/p7/variants/left/meshes/L3_Link.STL; visual mesh filename=../../components/arms/p7/variants/left/meshes/L3_Link.STL
- link arm_left_L4_Link: geometry collision mesh filename=../../components/arms/p7/variants/left/meshes/L4_Link.STL; visual mesh filename=../../components/arms/p7/variants/left/meshes/L4_Link.STL
- link arm_left_L5_Link: geometry collision mesh filename=../../components/arms/p7/variants/left/meshes/L5_Link.STL; visual mesh filename=../../components/arms/p7/variants/left/meshes/L5_Link.STL
- link arm_left_L6_Link: geometry collision mesh filename=../../components/arms/p7/variants/left/meshes/L6_Link.STL; visual mesh filename=../../components/arms/p7/variants/left/meshes/L6_Link.STL
- link arm_left_L7_Link: geometry collision mesh filename=../../components/arms/p7/variants/left/meshes/L7_Link.STL; visual mesh filename=../../components/arms/p7/variants/left/meshes/L7_Link.STL
- link arm_left_L8_Link: geometry collision mesh filename=../../components/arms/p7/variants/left/meshes/L8_Link.STL; visual mesh filename=../../components/arms/p7/variants/left/meshes/L8_Link.STL
- link arm_right_R1_Link: geometry collision mesh filename=../../components/arms/p7/variants/right/meshes/R1_Link.STL; visual mesh filename=../../components/arms/p7/variants/right/meshes/R1_Link.STL
- link arm_right_R2_Link: geometry collision mesh filename=../../components/arms/p7/variants/right/meshes/R2_Link.STL; visual mesh filename=../../components/arms/p7/variants/right/meshes/R2_Link.STL
- link arm_right_R3_Link: geometry collision mesh filename=../../components/arms/p7/variants/right/meshes/R3_Link.STL; visual mesh filename=../../components/arms/p7/variants/right/meshes/R3_Link.STL
- link arm_right_R4_Link: geometry collision mesh filename=../../components/arms/p7/variants/right/meshes/R4_Link.STL; visual mesh filename=../../components/arms/p7/variants/right/meshes/R4_Link.STL
- link arm_right_R5_Link: geometry collision mesh filename=../../components/arms/p7/variants/right/meshes/R5_Link.STL; visual mesh filename=../../components/arms/p7/variants/right/meshes/R5_Link.STL
- link arm_right_R6_Link: geometry collision mesh filename=../../components/arms/p7/variants/right/meshes/R6_Link.STL; visual mesh filename=../../components/arms/p7/variants/right/meshes/R6_Link.STL
- link arm_right_R7_Link: geometry collision mesh filename=../../components/arms/p7/variants/right/meshes/R7_Link.STL; visual mesh filename=../../components/arms/p7/variants/right/meshes/R7_Link.STL
- link arm_right_R8_Link: geometry collision mesh filename=../../components/arms/p7/variants/right/meshes/R8_Link.STL; visual mesh filename=../../components/arms/p7/variants/right/meshes/R8_Link.STL
- link base_base_link: geometry collision mesh filename=../../components/bases/p7_torso/variants/default/meshes/bas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; visual mesh filename=../../components/bases/p7_torso/variants/default/meshes/bas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

File: src/linker_robot_assets/assets/workstations/p7_i1_l25_bimanual/workstation.urdf (robot description, URDF)
Before this commit: robot lkls73_i1_l25_bimanual, 67 links, 66 joints
Links:
- link arm_left_L1_Link: geometry collision mesh filename=../../components/arms/p7/variants/left/meshes/L1_Link.STL; visual mesh filename=../../components/arms/p7/variants/left/meshes/L1_Link.STL
- link arm_left_L2_Link: geometry collision mesh filename=../../components/arms/p7/variants/left/meshes/L2_Link.STL; visual mesh filename=../../components/arms/p7/variants/left/meshes/L2_Link.STL
- link arm_left_L3_Link: geometry collision mesh filename=../../components/arms/p7/variants/left/meshes/L3_Link.STL; visual mesh filename=../../components/arms/p7/variants/left/meshes/L3_Link.STL
- link arm_left_L4_Link: geometry collision mesh filename=../../components/arms/p7/variants/left/meshes/L4_Link.STL; visual mesh filename=../../components/arms/p7/variants/left/meshes/L4_Link.STL
- link arm_left_L5_Link: geometry collision mesh filename=../../components/arms/p7/variants/left/meshes/L5_Link.STL; visual mesh filename=../../components/arms/p7/variants/left/meshes/L5_Link.STL
- link arm_left_L6_Link: geometry collision mesh filename=../../components/arms/p7/variants/left/meshes/L6_Link.STL; visual mesh filename=../../components/arms/p7/variants/left/meshes/L6_Link.STL
- link arm_left_L7_Link: geometry collision mesh filename=../../components/arms/p7/variants/left/meshes/L7_Link.STL; visual mesh filename=../../components/arms/p7/variants/left/meshes/L7_Link.STL
- link arm_left_L8_Link: geometry collision mesh filename=../../components/arms/p7/variants/left/meshes/L8_Link.STL; visual mesh filename=../../components/arms/p7/variants/left/meshes/L8_Link.STL
- link arm_right_R1_Link: geometry collision mesh filename=../../components/arms/p7/variants/right/meshes/R1_Link.STL; visual mesh filename=../../components/arms/p7/variants/right/meshes/R1_Link.STL
- link arm_right_R2_Link: geometry collision mesh filename=../../components/arms/p7/variants/right/meshes/R2_Link.STL; visual mesh filename=../../components/arms/p7/variants/right/meshes/R2_Link.STL
- link arm_right_R3_Link: geometry collision mesh filename=../../components/arms/p7/variants/right/meshes/R3_Link.STL; visual mesh filename=../../components/arms/p7/variants/right/meshes/R3_Link.STL
- link arm_right_R4_Link: geometry collision mesh filename=../../components/arms/p7/variants/right/meshes/R4_Link.STL; visual mesh filename=../../components/arms/p7/variants/right/meshes/R4_Link.STL
- link arm_right_R5_Link: geometry collision mesh filename=../../components/arms/p7/variants/right/meshes/R5_Link.STL; visual mesh filename=../../components/arms/p7/variants/right/meshes/R5_Link.STL
- link arm_right_R6_Link: geometry collision mesh filename=../../components/arms/p7/variants/right/meshes/R6_Link.STL; visual mesh filename=../../components/arms/p7/variants/right/meshes/R6_Link.STL
- link arm_right_R7_Link: geometry collision mesh filename=../../components/arms/p7/variants/right/meshes/R7_Link.STL; visual mesh filename=../../components/arms/p7/variants/right/meshes/R7_Link.STL
- link arm_right_R8_Link: geometry collision mesh filename=../../components/arms/p7/variants/right/meshes/R8_Link.STL; visual mesh filename=../../components/arms/p7/variants/right/meshes/R8_Link.STL
- link base_base_link: geometry collision mesh filename=../../components/bases/p7_torso/variants/default/meshes/bas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; visual mesh filename=../../components/bases/p7_torso/variants/default/meshes/bas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

File: src/linker_robot_assets/assets/workstations/p7_i1_o6_bimanual/workstation.urdf (robot description, URDF)
Before this commit: robot lkls73_i1_o6_bimanual, 47 links, 46 joints
Links:
- link arm_left_L1_Link: geometry collision mesh filename=../../components/arms/p7/variants/left/meshes/L1_Link.STL; visual mesh filename=../../components/arms/p7/variants/left/meshes/L1_Link.STL
- link arm_left_L2_Link: geometry collision mesh filename=../../components/arms/p7/variants/left/meshes/L2_Link.STL; visual mesh filename=../../components/arms/p7/variants/left/meshes/L2_Link.STL
- link arm_left_L3_Link: geometry collision mesh filename=../../components/arms/p7/variants/left/meshes/L3_Link.STL; visual mesh filename=../../components/arms/p7/variants/left/meshes/L3_Link.STL
- link arm_left_L4_Link: geometry collision mesh filename=../../components/arms/p7/variants/left/meshes/L4_Link.STL; visual mesh filename=../../components/arms/p7/variants/left/meshes/L4_Link.STL
- link arm_left_L5_Link: geometry collision mesh filename=../../components/arms/p7/variants/left/meshes/L5_Link.STL; visual mesh filename=../../components/arms/p7/variants/left/meshes/L5_Link.STL
- link arm_left_L6_Link: geometry collision mesh filename=../../components/arms/p7/variants/left/meshes/L6_Link.STL; visual mesh filename=../../components/arms/p7/variants/left/meshes/L6_Link.STL
- link arm_left_L7_Link: geometry collision mesh filename=../../components/arms/p7/variants/left/meshes/L7_Link.STL; visual mesh filename=../../components/arms/p7/variants/left/meshes/L7_Link.STL
- link arm_left_L8_Link: geometry collision mesh filename=../../components/arms/p7/variants/left/meshes/L8_Link.STL; visual mesh filename=../../components/arms/p7/variants/left/meshes/L8_Link.STL
- link arm_right_R1_Link: geometry collision mesh filename=../../components/arms/p7/variants/right/meshes/R1_Link.STL; visual mesh filename=../../components/arms/p7/variants/right/meshes/R1_Link.STL
- link arm_right_R2_Link: geometry collision mesh filename=../../components/arms/p7/variants/right/meshes/R2_Link.STL; visual mesh filename=../../components/arms/p7/variants/right/meshes/R2_Link.STL
- link arm_right_R3_Link: geometry collision mesh filename=../../components/arms/p7/variants/right/meshes/R3_Link.STL; visual mesh filename=../../components/arms/p7/variants/right/meshes/R3_Link.STL
- link arm_right_R4_Link: geometry collision mesh filename=../../components/arms/p7/variants/right/meshes/R4_Link.STL; visual mesh filename=../../components/arms/p7/variants/right/meshes/R4_Link.STL
- link arm_right_R5_Link: geometry collision mesh filename=../../components/arms/p7/variants/right/meshes/R5_Link.STL; visual mesh filename=../../components/arms/p7/variants/right/meshes/R5_Link.STL
- link arm_right_R6_Link: geometry collision mesh filename=../../components/arms/p7/variants/right/meshes/R6_Link.STL; visual mesh filename=../../components/arms/p7/variants/right/meshes/R6_Link.STL
- link arm_right_R7_Link: geometry collision mesh filename=../../components/arms/p7/variants/right/meshes/R7_Link.STL; visual mesh filename=../../components/arms/p7/variants/right/meshes/R7_Link.STL
- link arm_right_R8_Link: geometry collision mesh filename=../../components/arms/p7/variants/right/meshes/R8_Link.STL; visual mesh filename=../../components/arms/p7/variants/right/meshes/R8_Link.STL
- link base_base_link: geometry collision mesh filename=../../components/bases/p7_torso/variants/default/meshes/bas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; visual mesh filename=../../components/bases/p7_torso/variants/default/meshes/bas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
