Commit message: fix(arm): upright ar5_08 base convention; revert joint-dynamics strip
Two corrections to the Isaac-adoption asset work:

1. The Isaac arm instability was the base convention, not joint dynamics.
   ar5_08 baked a -90°X into joint_1's origin and its base geoms (arm rested
   horizontal +Y); Isaac's AR5V2 rests vertical (+Z, all origins rpy=0). The
   arms are otherwise identical (same joint origins, link inertias, joint-space
   mass matrix), but the horizontal rest pose destabilized the imported PhysX
   articulation under Isaac's stiff drive. Zero the -90°X on the ar5_08 base
   visual/collision geoms and joint_1 origin (both variants) so the composed
   arm rests upright: flange [0,0,0.8745] identity at qpos=0, M unchanged.

2. Revert the native joint-dynamics strip from the previous change. Removing
   intrinsic damping/armature/frictionloss was a misdiagnosis — it didn't fix
   the drift (the base convention did) and deleted real hardware modeling that
   MuJoCo/mujoco-wasm passive replay relies on. Isaac's runtime DriveAPI adds
   its damping on top of the joint's own; the intrinsic values are kept.

Composer now applies only the motor-actuator and placeholder-inertial
transforms. Changes ar5_08's rest orientation (horizontal -> vertical)
everywhere it's used; linker-sim / viser scenes need a root_pose re-orient.
Drift-clean and validate_workstation pass for all 23 workstations.

File: src/linker_robot_assets/assets/components/arms/ar5_08/variants/left/arm.urdf (robot description, URDF)
Before this commit: robot arm, 9 links, 8 joints
Joints:
- joint AR5_5_08L_W4C4A6_joint_1: origin xyz=0.0 0.0 0.0 rpy=-1.5708 0 0 -> xyz=0.0 0.0 0.0 rpy=0 0 0

File: src/linker_robot_assets/assets/components/arms/ar5_08/variants/right/arm.urdf (robot description, URDF)
Before this commit: robot arm, 9 links, 8 joints
Joints:
- joint AR5_5_08R_W4C4A6_joint_1: origin xyz=0.0 0.0 0.0 rpy=1.5708 0 0 -> xyz=0.0 0.0 0.0 rpy=0 0 0

File: src/linker_robot_assets/assets/workstations/ar5_08_l25_bench_bimanual/workstation.urdf (robot description, URDF)
Before this commit: robot ar5_08_l25_bench_bimanual, 68 links, 67 joints
Joints:
- joint arm_left_AR5_5_08L_W4C4A6_joint_1: origin xyz=0 0 0 rpy=-1.5708 0 0 -> xyz=0 0 0 rpy=0 0 0
- joint arm_right_AR5_5_08R_W4C4A6_joint_1: origin xyz=0 0 0 rpy=1.5708 0 0 -> xyz=0 0 0 rpy=0 0 0

File: src/linker_robot_assets/assets/workstations/ar5_08_l6_l/workstation.urdf (robot description, URDF)
Before this commit: robot ar5_08_l6_l, 27 links, 26 joints
Joints:
- joint arm_AR5_5_08L_W4C4A6_joint_1: origin xyz=0 0 0 rpy=-1.5708 0 0 -> xyz=0 0 0 rpy=0 0 0

File: src/linker_robot_assets/assets/workstations/ar5_08_l6_r/workstation.urdf (robot description, URDF)
Before this commit: robot ar5_08_l6_r, 27 links, 26 joints
Joints:
- joint arm_AR5_5_08R_W4C4A6_joint_1: origin xyz=0 0 0 rpy=1.5708 0 0 -> xyz=0 0 0 rpy=0 0 0

File: src/linker_robot_assets/assets/workstations/ar5_08_o6_bench_bimanual/workstation.urdf (robot description, URDF)
Before this commit: robot ar5_08_o6_bench_bimanual, 48 links, 47 joints
Joints:
- joint arm_left_AR5_5_08L_W4C4A6_joint_1: origin xyz=0 0 0 rpy=-1.5708 0 0 -> xyz=0 0 0 rpy=0 0 0
- joint arm_right_AR5_5_08R_W4C4A6_joint_1: origin xyz=0 0 0 rpy=1.5708 0 0 -> xyz=0 0 0 rpy=0 0 0

File: src/linker_robot_assets/assets/workstations/ar5_08_single_l/workstation.urdf (robot description, URDF)
Before this commit: robot ar5_08_single_l, 10 links, 9 joints
Joints:
- joint arm_AR5_5_08L_W4C4A6_joint_1: origin xyz=0 0 0 rpy=-1.5708 0 0 -> xyz=0 0 0 rpy=0 0 0

File: src/linker_robot_assets/assets/workstations/ar5_08_single_r/workstation.urdf (robot description, URDF)
Before this commit: robot ar5_08_single_r, 10 links, 9 joints
Joints:
- joint arm_AR5_5_08R_W4C4A6_joint_1: origin xyz=0 0 0 rpy=1.5708 0 0 -> xyz=0 0 0 rpy=0 0 0
