Commit message: fix(assets): correct ar5_08 bench mounts (stale upright-compensation + wrong hand)
ar5_08_{o6,l25}_bench_bimanual kept pre-v0.2.0 compensation: the arm base_mount
still rotated [±1.5708,0,∓1.5708] (to un-rotate an arm that is now upright) and
the hand wrist_mount used [3.1416,0,∓1.5708] / z=-0.038. Reset base_mount to
identity (matching the ar5(07) benches, same bench_table pads + upright arm) and
correct the hand mount to the ar5_08_l6 convention (rpy [0,0,±1.5708]) with the
measured +20.5 mm Z flange offset. Recomposed; validate_workstation clean.

File: src/linker_robot_assets/assets/workstations/ar5_08_l25_bench_bimanual/workstation.urdf (robot description, URDF)
Before this commit: robot ar5_08_l25_bench_bimanual, 68 links, 67 joints
Joints:
- joint mount_arm_left_to_base_base_mount: origin xyz=0 0 0 rpy=1.5708 0 -1.5708 -> xyz=0 0 0 rpy=0 0 0
- joint mount_arm_right_to_base_base_mount: origin xyz=0 0 0 rpy=-1.5708 0 1.5708 -> xyz=0 0 0 rpy=0 0 0
- joint mount_hand_left_to_arm_left_wrist_mount: origin xyz=0 0 -0.038 rpy=3.1416 0 -1.5708 -> xyz=0 0 0.0205 rpy=0 0 1.5708
- joint mount_hand_right_to_arm_right_wrist_mount: origin xyz=0 0 -0.038 rpy=3.1416 0 1.5708 -> xyz=0 0 0.0205 rpy=0 0 -1.5708

File: src/linker_robot_assets/assets/workstations/ar5_08_o6_bench_bimanual/workstation.urdf (robot description, URDF)
Before this commit: robot ar5_08_o6_bench_bimanual, 48 links, 47 joints
Joints:
- joint mount_arm_left_to_base_base_mount: origin xyz=0 0 0 rpy=1.5708 0 -1.5708 -> xyz=0 0 0 rpy=0 0 0
- joint mount_arm_right_to_base_base_mount: origin xyz=0 0 0 rpy=-1.5708 0 1.5708 -> xyz=0 0 0 rpy=0 0 0
- joint mount_hand_left_to_arm_left_wrist_mount: origin xyz=0 0 -0.038 rpy=3.1416 0 -1.5708 -> xyz=0 0 0.0205 rpy=0 0 1.5708
- joint mount_hand_right_to_arm_right_wrist_mount: origin xyz=0 0 -0.038 rpy=3.1416 0 1.5708 -> xyz=0 0 0.0205 rpy=0 0 -1.5708
