Commit message: fix(assets): mirror the L25 right-hand finger roll axes
The L25 hand variants are mirrored across y=0 -- every finger's mcp_roll
origin has its y negated between sides. Under that reflection a rotation
axis transforms as a pseudovector, (ax, ay, az) -> (-ax, ay, -az), so the
right variant's four finger roll axes should be the negation of the left's.
They were copied verbatim as "-1 0 0" instead.

Consequence: for the same joint value, all four fingers abducted toward the
pinky side on the left hand but toward the index side on the right -- the
right hand's abduction ran backwards versus the physical robot. Confirmed by
eyeballing a per-joint sweep recording (episode_000015) against hardware.

The thumb was already correct (thumb_cmc_roll and thumb_cmc_yaw are both
mirrored), and *_mcp_pitch is correctly identical on both sides because the
mirror preserves the y component -- which is why only the rolls were wrong.
linkerhand_l20lite mirrors its finger rolls correctly and is the in-tree
precedent for the rule.

Fix flips the four axes in the right variant's hand.urdf and hand.mjcf, and
re-composes the 5 l25 workstations plus the l25_r / ar5_08_l25_r units.
check_drift.sh is clean; joint names are unchanged, so no rename semver
concern. Verified by FK on both the component and the composed workstation:
fingertip displacement at roll=+max is now exactly negated between sides in
each hand's own frame (+-17.21mm index, +-17.44mm others).

Note this changes geometry, not decoded values: decode_hand still maps the
same SDK count to the same joint angle. Anything consuming right-hand roll
joint *values* now gets the mirrored physical motion for those values.

linkerhand_l30 has the identical un-mirrored axes but no workstation or unit
references it; left untouched and unvalidated (no L30 hardware data).

File: src/linker_robot_assets/assets/components/hands/linkerhand_l25/variants/right/hand.urdf (robot description, URDF)
Before this commit: robot hand, 22 links, 21 joints
Joints:
- joint rh_index_mcp_roll: axis -1 0 0 -> 1 0 0
- joint rh_middle_mcp_roll: axis -1 0 0 -> 1 0 0
- joint rh_pinky_mcp_roll: axis -1 0 0 -> 1 0 0
- joint rh_ring_mcp_roll: axis -1 0 0 -> 1 0 0

File: src/linker_robot_assets/assets/units/ar5_08_l25_r/workstation.urdf (robot description, URDF)
Before this commit: robot ar5_08_l25_r, 32 links, 31 joints
Joints:
- joint hand_rh_index_mcp_roll: axis -1 0 0 -> 1 0 0
- joint hand_rh_middle_mcp_roll: axis -1 0 0 -> 1 0 0
- joint hand_rh_pinky_mcp_roll: axis -1 0 0 -> 1 0 0
- joint hand_rh_ring_mcp_roll: axis -1 0 0 -> 1 0 0

File: src/linker_robot_assets/assets/units/l25_r/workstation.urdf (robot description, URDF)
Before this commit: robot l25_r, 23 links, 22 joints
Joints:
- joint hand_rh_index_mcp_roll: axis -1 0 0 -> 1 0 0
- joint hand_rh_middle_mcp_roll: axis -1 0 0 -> 1 0 0
- joint hand_rh_pinky_mcp_roll: axis -1 0 0 -> 1 0 0
- joint hand_rh_ring_mcp_roll: axis -1 0 0 -> 1 0 0

File: src/linker_robot_assets/assets/workstations/a7_l25_dc/workstation.urdf (robot description, URDF)
Before this commit: robot a7_l25_dc, 65 links, 64 joints
Joints:
- joint hand_right_rh_index_mcp_roll: axis -1 0 0 -> 1 0 0
- joint hand_right_rh_middle_mcp_roll: axis -1 0 0 -> 1 0 0
- joint hand_right_rh_pinky_mcp_roll: axis -1 0 0 -> 1 0 0
- joint hand_right_rh_ring_mcp_roll: axis -1 0 0 -> 1 0 0

File: src/linker_robot_assets/assets/workstations/a7_lite_l25_dc/workstation.urdf (robot description, URDF)
Before this commit: robot a7_lite_l25_dc, 65 links, 64 joints
Joints:
- joint hand_right_rh_index_mcp_roll: axis -1 0 0 -> 1 0 0
- joint hand_right_rh_middle_mcp_roll: axis -1 0 0 -> 1 0 0
- joint hand_right_rh_pinky_mcp_roll: axis -1 0 0 -> 1 0 0
- joint hand_right_rh_ring_mcp_roll: axis -1 0 0 -> 1 0 0

File: src/linker_robot_assets/assets/workstations/ar5_08_l25_bench_bimanual/workstation.urdf (robot description, URDF)
Before this commit: robot ar5_08_l25_bench_bimanual, 68 links, 67 joints
Joints:
- joint hand_right_rh_index_mcp_roll: axis -1 0 0 -> 1 0 0
- joint hand_right_rh_middle_mcp_roll: axis -1 0 0 -> 1 0 0
- joint hand_right_rh_pinky_mcp_roll: axis -1 0 0 -> 1 0 0
- joint hand_right_rh_ring_mcp_roll: axis -1 0 0 -> 1 0 0

File: src/linker_robot_assets/assets/workstations/ar5_l25_bench_bimanual/workstation.urdf (robot description, URDF)
Before this commit: robot ar5_l25_bench_bimanual, 68 links, 67 joints
Joints:
- joint hand_right_rh_index_mcp_roll: axis -1 0 0 -> 1 0 0
- joint hand_right_rh_middle_mcp_roll: axis -1 0 0 -> 1 0 0
- joint hand_right_rh_pinky_mcp_roll: axis -1 0 0 -> 1 0 0
- joint hand_right_rh_ring_mcp_roll: axis -1 0 0 -> 1 0 0

File: src/linker_robot_assets/assets/workstations/p7_i1_l25_bimanual/workstation.urdf (robot description, URDF)
Before this commit: robot p7_i1_l25_bimanual, 67 links, 66 joints
Joints:
- joint hand_right_rh_index_mcp_roll: axis -1 0 0 -> 1 0 0
- joint hand_right_rh_middle_mcp_roll: axis -1 0 0 -> 1 0 0
- joint hand_right_rh_pinky_mcp_roll: axis -1 0 0 -> 1 0 0
- joint hand_right_rh_ring_mcp_roll: axis -1 0 0 -> 1 0 0
