Commit message: fix(assets): restore collision checks outside mounting seams
Use explicit, documented body-pair exclusions and preserve structural openings in base colliders. Regenerate assets on the latest main while retaining the L25 right-hand axis correction.

Refs linker-bot/linker-sim-isaac#28

File: src/linker_robot_assets/assets/components/bases/a7_lite_torso/variants/default/base.urdf (robot description, URDF)
Before this commit: robot a7_lite_torso, 4 links, 3 joints
Links:
- link base_link: geometry collision mesh filename=meshes/collision/base_part_000.stl; collision mesh filename=meshes/collision/base_part_001.stl

File: src/linker_robot_assets/assets/components/bases/a7_torso/variants/default/base.urdf (robot description, URDF)
Before this commit: robot a7_torso, 4 links, 3 joints
Links:
- link base_link: geometry collision mesh filename=meshes/collision/base_part_000.stl; collision mesh filename=meshes/collision/base_part_001.stl

File: src/linker_robot_assets/assets/components/bases/bench_table/variants/default/base.urdf (robot description, URDF)
Before this commit: robot workstation, 5 links, 4 joints
Links:
- link workstation_link: geometry collision mesh filename=meshes/collision/base_part_000.stl; collision mesh filename=meshes/collision/base_part_001.stl

File: src/linker_robot_assets/assets/components/bases/p7_torso/variants/default/base.urdf (robot description, URDF)
Before this commit: robot p7_torso, 4 links, 3 joints
Links:
- link base_link: geometry collision mesh filename=meshes/collision/base_part_000.stl; collision mesh filename=meshes/collision/base_part_001.stl

File: src/linker_robot_assets/assets/workstations/a7_l20lite_dc/workstation.urdf (robot description, URDF)
Before this commit: robot a7_l20lite_dc, 63 links, 62 joints
Links:
- link base_base_link: geometry collision mesh filename=../../components/bases/a7_torso/variants/default/meshes/col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; collision mesh filename=../../components/bases/a7_torso/variants/default/meshes/col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

File: src/linker_robot_assets/assets/workstations/a7_l25_dc/workstation.urdf (robot description, URDF)
Before this commit: robot a7_l25_dc, 65 links, 64 joints
Links:
- link base_base_link: geometry collision mesh filename=../../components/bases/a7_torso/variants/default/meshes/col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; collision mesh filename=../../components/bases/a7_torso/variants/default/meshes/col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

File: src/linker_robot_assets/assets/workstations/a7_l6_dc/workstation.urdf (robot description, URDF)
Before this commit: robot a7_l6_dc, 55 links, 54 joints
Links:
- link base_base_link: geometry collision mesh filename=../../components/bases/a7_torso/variants/default/meshes/col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; collision mesh filename=../../components/bases/a7_torso/variants/default/meshes/col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

File: src/linker_robot_assets/assets/workstations/a7_lite_l20lite_dc/workstation.urdf (robot description, URDF)
Before this commit: robot a7_lite_l20lite_dc, 63 links, 62 joints
Links:
- link base_base_link: geometry collision mesh filename=../../components/bases/a7_lite_torso/variants/default/meshe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; collision mesh filename=../../components/bases/a7_lite_torso/variants/default/meshe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

File: src/linker_robot_assets/assets/workstations/a7_lite_l25_dc/workstation.urdf (robot description, URDF)
Before this commit: robot a7_lite_l25_dc, 65 links, 64 joints
Links:
- link base_base_link: geometry collision mesh filename=../../components/bases/a7_lite_torso/variants/default/meshe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; collision mesh filename=../../components/bases/a7_lite_torso/variants/default/meshe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

File: src/linker_robot_assets/assets/workstations/a7_lite_l6_dc/workstation.urdf (robot description, URDF)
Before this commit: robot a7_lite_l6_dc, 55 links, 54 joints
Links:
- link base_base_link: geometry collision mesh filename=../../components/bases/a7_lite_torso/variants/default/meshe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; collision mesh filename=../../components/bases/a7_lite_torso/variants/default/meshe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

File: src/linker_robot_assets/assets/workstations/a7_lite_o6_dc/workstation.urdf (robot description, URDF)
Before this commit: robot a7_lite_o6_dc, 45 links, 44 joints
Links:
- link base_base_link: geometry collision mesh filename=../../components/bases/a7_lite_torso/variants/default/meshe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; collision mesh filename=../../components/bases/a7_lite_torso/variants/default/meshe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

File: src/linker_robot_assets/assets/workstations/a7_o6_dc/workstation.urdf (robot description, URDF)
Before this commit: robot a7_o6_dc, 45 links, 44 joints
Links:
- link base_base_link: geometry collision mesh filename=../../components/bases/a7_torso/variants/default/meshes/col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; collision mesh filename=../../components/bases/a7_torso/variants/default/meshes/col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

File: src/linker_robot_assets/assets/workstations/ar5_08_l25_bench_bimanual/workstation.urdf (robot description, URDF)
Before this commit: robot ar5_08_l25_bench_bimanual, 68 links, 67 joints
Links:
- link base_workstation_link: geometry collision mesh filename=../../components/bases/bench_table/variants/default/meshes/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; collision mesh filename=../../components/bases/bench_table/variants/default/meshes/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

File: src/linker_robot_assets/assets/workstations/ar5_08_o6_bench_bimanual/workstation.urdf (robot description, URDF)
Before this commit: robot ar5_08_o6_bench_bimanual, 48 links, 47 joints
Links:
- link base_workstation_link: geometry collision mesh filename=../../components/bases/bench_table/variants/default/meshes/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; collision mesh filename=../../components/bases/bench_table/variants/default/meshes/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

File: src/linker_robot_assets/assets/workstations/ar5_l25_bench_bimanual/workstation.urdf (robot description, URDF)
Before this commit: robot ar5_l25_bench_bimanual, 68 links, 67 joints
Links:
- link base_workstation_link: geometry collision mesh filename=../../components/bases/bench_table/variants/default/meshes/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; collision mesh filename=../../components/bases/bench_table/variants/default/meshes/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

File: src/linker_robot_assets/assets/workstations/ar5_l6_bench_bimanual/workstation.urdf (robot description, URDF)
Before this commit: robot ar5_l6_bench_bimanual, 58 links, 57 joints
Links:
- link base_workstation_link: geometry collision mesh filename=../../components/bases/bench_table/variants/default/meshes/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; collision mesh filename=../../components/bases/bench_table/variants/default/meshes/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

File: src/linker_robot_assets/assets/workstations/ar5_o6_bench_bimanual/workstation.urdf (robot description, URDF)
Before this commit: robot ar5_o6_bench_bimanual, 48 links, 47 joints
Links:
- link base_workstation_link: geometry collision mesh filename=../../components/bases/bench_table/variants/default/meshes/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; collision mesh filename=../../components/bases/bench_table/variants/default/meshes/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

File: src/linker_robot_assets/assets/workstations/p7_i1_l20lite_bimanual/workstation.urdf (robot description, URDF)
Before this commit: robot p7_i1_l20lite_bimanual, 65 links, 64 joints
Links:
- link base_base_link: geometry collision mesh filename=../../components/bases/p7_torso/variants/default/meshes/col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; collision mesh filename=../../components/bases/p7_torso/variants/default/meshes/col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

File: src/linker_robot_assets/assets/workstations/p7_i1_l25_bimanual/workstation.urdf (robot description, URDF)
Before this commit: robot p7_i1_l25_bimanual, 67 links, 66 joints
Links:
- link base_base_link: geometry collision mesh filename=../../components/bases/p7_torso/variants/default/meshes/col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; collision mesh filename=../../components/bases/p7_torso/variants/default/meshes/col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

File: src/linker_robot_assets/assets/workstations/p7_i1_l6_bimanual/workstation.urdf (robot description, URDF)
Before this commit: robot p7_i1_l6_bimanual, 57 links, 56 joints
Links:
- link base_base_link: geometry collision mesh filename=../../components/bases/p7_torso/variants/default/meshes/col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; collision mesh filename=../../components/bases/p7_torso/variants/default/meshes/col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

Commit message: refactor(assets): group base colliders by physical assemblies

File: src/linker_robot_assets/assets/components/bases/a7_lite_torso/variants/default/base.urdf (robot description, URDF)
Before this commit: robot a7_lite_torso, 4 links, 3 joints
Links:
- link base_link: geometry collision box size=0.000100001478467754 0.0109668258938048 0.0360740187263812; collision box size=0.00010000158958734 0.0116303856029182 0.0294109775901053

File: src/linker_robot_assets/assets/components/bases/a7_torso/variants/default/base.urdf (robot description, URDF)
Before this commit: robot a7_torso, 4 links, 3 joints
Links:
- link base_link: geometry collision box size=0.0168008918408304 0.00300748646259308 0.00473126769065857; collision box size=0.0502374065108597 0.00513970106840134 0.0118521898984909

File: src/linker_robot_assets/assets/components/bases/bench_table/variants/default/base.urdf (robot description, URDF)
Before this commit: robot workstation, 5 links, 4 joints
Links:
- link workstation_link: geometry collision box size=0.059999942779541 0.120000123977661 1.08000007271767; collision box size=0.0599999949336052 0.0599999874830246 0.0115000009536743

File: src/linker_robot_assets/assets/components/bases/p7_torso/variants/default/base.urdf (robot description, URDF)
Before this commit: robot p7_torso, 4 links, 3 joints
Links:
- link base_link: geometry collision box size=0.000255171961484821 0.00555124425806092 0.0449999570846558; collision box size=0.000255171961484828 0.00555124425806086 0.0449999570846558

File: src/linker_robot_assets/assets/workstations/a7_l20lite_dc/workstation.urdf (robot description, URDF)
Before this commit: robot a7_l20lite_dc, 63 links, 62 joints
Links:
- link base_base_link: geometry collision box size=0.0168008918 0.00300748646 0.00473126769; collision box size=0.0502374065 0.00513970107 0.0118521899

File: src/linker_robot_assets/assets/workstations/a7_l25_dc/workstation.urdf (robot description, URDF)
Before this commit: robot a7_l25_dc, 65 links, 64 joints
Links:
- link base_base_link: geometry collision box size=0.0168008918 0.00300748646 0.00473126769; collision box size=0.0502374065 0.00513970107 0.0118521899

File: src/linker_robot_assets/assets/workstations/a7_l6_dc/workstation.urdf (robot description, URDF)
Before this commit: robot a7_l6_dc, 55 links, 54 joints
Links:
- link base_base_link: geometry collision box size=0.0168008918 0.00300748646 0.00473126769; collision box size=0.0502374065 0.00513970107 0.0118521899

File: src/linker_robot_assets/assets/workstations/a7_lite_l20lite_dc/workstation.urdf (robot description, URDF)
Before this commit: robot a7_lite_l20lite_dc, 63 links, 62 joints
Links:
- link base_base_link: geometry collision box size=0.000100001478 0.0109668259 0.0360740187; collision box size=0.00010000159 0.0116303856 0.0294109776

File: src/linker_robot_assets/assets/workstations/a7_lite_l25_dc/workstation.urdf (robot description, URDF)
Before this commit: robot a7_lite_l25_dc, 65 links, 64 joints
Links:
- link base_base_link: geometry collision box size=0.000100001478 0.0109668259 0.0360740187; collision box size=0.00010000159 0.0116303856 0.0294109776

File: src/linker_robot_assets/assets/workstations/a7_lite_l6_dc/workstation.urdf (robot description, URDF)
Before this commit: robot a7_lite_l6_dc, 55 links, 54 joints
Links:
- link base_base_link: geometry collision box size=0.000100001478 0.0109668259 0.0360740187; collision box size=0.00010000159 0.0116303856 0.0294109776

File: src/linker_robot_assets/assets/workstations/a7_lite_o6_dc/workstation.urdf (robot description, URDF)
Before this commit: robot a7_lite_o6_dc, 45 links, 44 joints
Links:
- link base_base_link: geometry collision box size=0.000100001478 0.0109668259 0.0360740187; collision box size=0.00010000159 0.0116303856 0.0294109776

File: src/linker_robot_assets/assets/workstations/a7_o6_dc/workstation.urdf (robot description, URDF)
Before this commit: robot a7_o6_dc, 45 links, 44 joints
Links:
- link base_base_link: geometry collision box size=0.0168008918 0.00300748646 0.00473126769; collision box size=0.0502374065 0.00513970107 0.0118521899

File: src/linker_robot_assets/assets/workstations/ar5_08_l25_bench_bimanual/workstation.urdf (robot description, URDF)
Before this commit: robot ar5_08_l25_bench_bimanual, 68 links, 67 joints
Links:
- link base_workstation_link: geometry collision box size=0.0599999428 0.120000124 1.08000007; collision box size=0.0599999949 0.0599999875 0.011500001

File: src/linker_robot_assets/assets/workstations/ar5_08_o6_bench_bimanual/workstation.urdf (robot description, URDF)
Before this commit: robot ar5_08_o6_bench_bimanual, 48 links, 47 joints
Links:
- link base_workstation_link: geometry collision box size=0.0599999428 0.120000124 1.08000007; collision box size=0.0599999949 0.0599999875 0.011500001

File: src/linker_robot_assets/assets/workstations/ar5_l25_bench_bimanual/workstation.urdf (robot description, URDF)
Before this commit: robot ar5_l25_bench_bimanual, 68 links, 67 joints
Links:
- link base_workstation_link: geometry collision box size=0.0599999428 0.120000124 1.08000007; collision box size=0.0599999949 0.0599999875 0.011500001

File: src/linker_robot_assets/assets/workstations/ar5_l6_bench_bimanual/workstation.urdf (robot description, URDF)
Before this commit: robot ar5_l6_bench_bimanual, 58 links, 57 joints
Links:
- link base_workstation_link: geometry collision box size=0.0599999428 0.120000124 1.08000007; collision box size=0.0599999949 0.0599999875 0.011500001

File: src/linker_robot_assets/assets/workstations/ar5_o6_bench_bimanual/workstation.urdf (robot description, URDF)
Before this commit: robot ar5_o6_bench_bimanual, 48 links, 47 joints
Links:
- link base_workstation_link: geometry collision box size=0.0599999428 0.120000124 1.08000007; collision box size=0.0599999949 0.0599999875 0.011500001

File: src/linker_robot_assets/assets/workstations/p7_i1_l20lite_bimanual/workstation.urdf (robot description, URDF)
Before this commit: robot p7_i1_l20lite_bimanual, 65 links, 64 joints
Links:
- link base_base_link: geometry collision box size=0.000255171961 0.00555124426 0.0449999571; collision box size=0.000255171961 0.00555124426 0.0449999571

File: src/linker_robot_assets/assets/workstations/p7_i1_l25_bimanual/workstation.urdf (robot description, URDF)
Before this commit: robot p7_i1_l25_bimanual, 67 links, 66 joints
Links:
- link base_base_link: geometry collision box size=0.000255171961 0.00555124426 0.0449999571; collision box size=0.000255171961 0.00555124426 0.0449999571

File: src/linker_robot_assets/assets/workstations/p7_i1_l6_bimanual/workstation.urdf (robot description, URDF)
Before this commit: robot p7_i1_l6_bimanual, 57 links, 56 joints
Links:
- link base_base_link: geometry collision box size=0.000255171961 0.00555124426 0.0449999571; collision box size=0.000255171961 0.00555124426 0.0449999571
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