Commit message: feat(assets): add shared flanges and optional camera assemblies

File: src/linker_robot_assets/assets/components/bases/bench_table/variants/default/base.urdf (robot description, URDF)
Before this commit: robot workstation, 5 links, 4 joints
Links:
- removed link camera
- removed link camera_base_link
- added link workstation_camera_mount
Joints:
- removed joint cameraBase
- removed joint cameraJoint
- added joint weld_workstation_camera_mount: type fixed, parent workstation_link, child workstation_camera_mount, origin xyz=0.0335 0.67 1.2974 rpy=-1.5708 0 -1.5708

File: src/linker_robot_assets/assets/units/ar5_08_l6_l/workstation.urdf (robot description, URDF)
Before this commit: robot ar5_08_l6_l, 27 links, 26 joints
Links:
- added link flange_flange_link, mass 0.044499999; collision mesh filename=../../components/attachments/ar5_08_l6_o6_flange/variants/d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; collision mesh filename=../../components/attachments/ar5_08_l6_o6_flange/variants/d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
- added link flange_hand_mount, mass 1e-09
Joints:
- removed joint mount_hand_to_arm_wrist_mount
- added joint flange_hand_mount_joint: type fixed, parent flange_flange_link, child flange_hand_mount, origin xyz=0 0 0.0225 rpy=0 0 0
- added joint mount_flange_to_arm_arm_mount: type fixed, parent arm_AR5_5_08L_W4C4A6_tcp, child flange_flange_link, origin xyz=0 0 0 rpy=0 0 -1.57079633
- added joint mount_hand_to_flange_wrist_mount: type fixed, parent flange_hand_mount, child hand_lh_hand_base_link, origin xyz=0 0 0 rpy=0 0 3.14159265

File: src/linker_robot_assets/assets/units/ar5_08_l6_r/workstation.urdf (robot description, URDF)
Before this commit: robot ar5_08_l6_r, 27 links, 26 joints
Links:
- added link flange_flange_link, mass 0.044499999; collision mesh filename=../../components/attachments/ar5_08_l6_o6_flange/variants/d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; collision mesh filename=../../components/attachments/ar5_08_l6_o6_flange/variants/d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
- added link flange_hand_mount, mass 1e-09
Joints:
- removed joint mount_hand_to_arm_wrist_mount
- added joint flange_hand_mount_joint: type fixed, parent flange_flange_link, child flange_hand_mount, origin xyz=0 0 0.0225 rpy=0 0 0
- added joint mount_flange_to_arm_arm_mount: type fixed, parent arm_AR5_5_08R_W4C4A6_tcp, child flange_flange_link, origin xyz=0 0 0 rpy=0 0 1.57079633
- added joint mount_hand_to_flange_wrist_mount: type fixed, parent flange_hand_mount, child hand_rh_hand_base_link, origin xyz=0 0 0 rpy=0.034906585 0 -3.14159265

File: src/linker_robot_assets/assets/units/ar5_08_o6_l/workstation.urdf (robot description, URDF)
Before this commit: robot ar5_08_o6_l, 22 links, 21 joints
Links:
- added link flange_flange_link, mass 0.044499999; collision mesh filename=../../components/attachments/ar5_08_l6_o6_flange/variants/d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; collision mesh filename=../../components/attachments/ar5_08_l6_o6_flange/variants/d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
- added link flange_hand_mount, mass 1e-09
Joints:
- removed joint mount_hand_to_arm_wrist_mount
- added joint flange_hand_mount_joint: type fixed, parent flange_flange_link, child flange_hand_mount, origin xyz=0 0 0.0225 rpy=0 0 0
- added joint mount_flange_to_arm_arm_mount: type fixed, parent arm_AR5_5_08L_W4C4A6_tcp, child flange_flange_link, origin xyz=0 0 0 rpy=0 0 -1.57079633
- added joint mount_hand_to_flange_wrist_mount: type fixed, parent flange_hand_mount, child hand_lh_hand_base_link, origin xyz=0 0 0 rpy=0 0 3.14159265

File: src/linker_robot_assets/assets/units/ar5_08_o6_r/workstation.urdf (robot description, URDF)
Before this commit: robot ar5_08_o6_r, 22 links, 21 joints
Links:
- added link flange_flange_link, mass 0.044499999; collision mesh filename=../../components/attachments/ar5_08_l6_o6_flange/variants/d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; collision mesh filename=../../components/attachments/ar5_08_l6_o6_flange/variants/d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
- added link flange_hand_mount, mass 1e-09
Joints:
- removed joint mount_hand_to_arm_wrist_mount
- added joint flange_hand_mount_joint: type fixed, parent flange_flange_link, child flange_hand_mount, origin xyz=0 0 0.0225 rpy=0 0 0
- added joint mount_flange_to_arm_arm_mount: type fixed, parent arm_AR5_5_08R_W4C4A6_tcp, child flange_flange_link, origin xyz=0 0 0 rpy=0 0 1.57079633
- added joint mount_hand_to_flange_wrist_mount: type fixed, parent flange_hand_mount, child hand_rh_hand_base_link, origin xyz=0 0 -0.002 rpy=0 0 -3.14159265

File: src/linker_robot_assets/assets/workstations/ar5_08_l25_bench_bimanual/workstation.urdf (robot description, URDF)
Before this commit: robot ar5_08_l25_bench_bimanual, 68 links, 67 joints
Links:
- removed link base_camera
- removed link base_camera_base_link
- added link base_workstation_camera_mount
- added link top_camera_camera, mass 0.170230156191785; collision mesh filename=../../components/sensors/workstation_zed2i/variants/default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; visual mesh filename=../../components/sensors/workstation_zed2i/variants/default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
- added link top_camera_camera_base_link, mass 0.120253078965696; collision mesh filename=../../components/sensors/workstation_zed2i/variants/default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; visual mesh filename=../../components/sensors/workstation_zed2i/variants/default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
- added link top_camera_left_optical, mass 1e-9
- added link top_camera_right_optical, mass 1e-9
Joints:
- removed joint base_cameraBase
- removed joint base_cameraJoint
- added joint base_weld_workstation_camera_mount: type fixed, parent base_workstation_link, child base_workstation_camera_mount, origin xyz=0.0335 0.67 1.2974 rpy=-1.5708 0 -1.5708
- added joint mount_top_camera_to_base_base_mount: type fixed, parent base_workstation_camera_mount, child top_camera_camera_base_link, origin xyz=0 0 0 rpy=0 0 0
- added joint top_camera_cameraJoint: type fixed, parent top_camera_camera_base_link, child top_camera_camera, origin xyz=0.0802 0.193139854 -0.275851476 rpy=-1.26599038 -0.643554018 -1.57079633, axis 0 0 0
- added joint top_camera_left_optical_joint: type fixed, parent top_camera_camera, child top_camera_left_optical, origin xyz=0.424482885 -0.150393718 -0.0524849102 rpy=-0.543269873 -1.26599038 1.57079633
- added joint top_camera_right_optical_joint: type fixed, parent top_camera_camera, child top_camera_right_optical, origin xyz=0.424482885 -0.114380749 0.0619837129 rpy=-0.543269873 -1.26599038 1.57079633

File: src/linker_robot_assets/assets/workstations/ar5_08_o6_bench_bimanual/workstation.urdf (robot description, URDF)
Before this commit: robot ar5_08_o6_bench_bimanual, 48 links, 47 joints
Links:
- removed link base_camera
- removed link base_camera_base_link
- added link base_workstation_camera_mount
- added link flange_left_flange_link, mass 0.044499999; collision mesh filename=../../components/attachments/ar5_08_l6_o6_flange/variants/d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; collision mesh filename=../../components/attachments/ar5_08_l6_o6_flange/variants/d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
- added link flange_left_hand_mount, mass 1e-09
- added link flange_right_flange_link, mass 0.044499999; collision mesh filename=../../components/attachments/ar5_08_l6_o6_flange/variants/d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; collision mesh filename=../../components/attachments/ar5_08_l6_o6_flange/variants/d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
- added link flange_right_hand_mount, mass 1e-09
- added link top_camera_camera, mass 0.170230156191785; collision mesh filename=../../components/sensors/workstation_zed2i/variants/default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; visual mesh filename=../../components/sensors/workstation_zed2i/variants/default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
- added link top_camera_camera_base_link, mass 0.120253078965696; collision mesh filename=../../components/sensors/workstation_zed2i/variants/default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; visual mesh filename=../../components/sensors/workstation_zed2i/variants/default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
- added link top_camera_left_optical, mass 1e-9
- added link top_camera_right_optical, mass 1e-9
Joints:
- removed joint base_cameraBase
- removed joint base_cameraJoint
- removed joint mount_hand_left_to_arm_left_wrist_mount
- removed joint mount_hand_right_to_arm_right_wrist_mount
- added joint base_weld_workstation_camera_mount: type fixed, parent base_workstation_link, child base_workstation_camera_mount, origin xyz=0.0335 0.67 1.2974 rpy=-1.5708 0 -1.5708
- added joint flange_left_hand_mount_joint: type fixed, parent flange_left_flange_link, child flange_left_hand_mount, origin xyz=0 0 0.0225 rpy=0 0 0
- added joint flange_right_hand_mount_joint: type fixed, parent flange_right_flange_link, child flange_right_hand_mount, origin xyz=0 0 0.0225 rpy=0 0 0
- added joint mount_flange_left_to_arm_left_arm_mount: type fixed, parent arm_left_AR5_5_08L_W4C4A6_tcp, child flange_left_flange_link, origin xyz=0 0 0 rpy=0 0 -1.57079633
- added joint mount_flange_right_to_arm_right_arm_mount: type fixed, parent arm_right_AR5_5_08R_W4C4A6_tcp, child flange_right_flange_link, origin xyz=0 0 0 rpy=0 0 1.57079633
- added joint mount_hand_left_to_flange_left_wrist_mount: type fixed, parent flange_left_hand_mount, child hand_left_lh_hand_base_link, origin xyz=0 0 0 rpy=0 0 3.14159265
- added joint mount_hand_right_to_flange_right_wrist_mount: type fixed, parent flange_right_hand_mount, child hand_right_rh_hand_base_link, origin xyz=0 0 -0.002 rpy=0 0 -3.14159265
- added joint mount_top_camera_to_base_base_mount: type fixed, parent base_workstation_camera_mount, child top_camera_camera_base_link, origin xyz=0 0 0 rpy=0 0 0
- added joint top_camera_cameraJoint: type fixed, parent top_camera_camera_base_link, child top_camera_camera, origin xyz=0.0802 0.193139854 -0.275851476 rpy=-1.26599038 -0.643554018 -1.57079633, axis 0 0 0
- added joint top_camera_left_optical_joint: type fixed, parent top_camera_camera, child top_camera_left_optical, origin xyz=0.424482885 -0.150393718 -0.0524849102 rpy=-0.543269873 -1.26599038 1.57079633
- added joint top_camera_right_optical_joint: type fixed, parent top_camera_camera, child top_camera_right_optical, origin xyz=0.424482885 -0.114380749 0.0619837129 rpy=-0.543269873 -1.26599038 1.57079633

File: src/linker_robot_assets/assets/workstations/ar5_l25_bench_bimanual/workstation.urdf (robot description, URDF)
Before this commit: robot ar5_l25_bench_bimanual, 68 links, 67 joints
Links:
- removed link base_camera
- removed link base_camera_base_link
- added link base_workstation_camera_mount
- added link top_camera_camera, mass 0.170230156191785; collision mesh filename=../../components/sensors/workstation_zed2i/variants/default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; visual mesh filename=../../components/sensors/workstation_zed2i/variants/default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
- added link top_camera_camera_base_link, mass 0.120253078965696; collision mesh filename=../../components/sensors/workstation_zed2i/variants/default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; visual mesh filename=../../components/sensors/workstation_zed2i/variants/default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
- added link top_camera_left_optical, mass 1e-9
- added link top_camera_right_optical, mass 1e-9
Joints:
- removed joint base_cameraBase
- removed joint base_cameraJoint
- added joint base_weld_workstation_camera_mount: type fixed, parent base_workstation_link, child base_workstation_camera_mount, origin xyz=0.0335 0.67 1.2974 rpy=-1.5708 0 -1.5708
- added joint mount_top_camera_to_base_base_mount: type fixed, parent base_workstation_camera_mount, child top_camera_camera_base_link, origin xyz=0 0 0 rpy=0 0 0
- added joint top_camera_cameraJoint: type fixed, parent top_camera_camera_base_link, child top_camera_camera, origin xyz=0.0802 0.193139854 -0.275851476 rpy=-1.26599038 -0.643554018 -1.57079633, axis 0 0 0
- added joint top_camera_left_optical_joint: type fixed, parent top_camera_camera, child top_camera_left_optical, origin xyz=0.424482885 -0.150393718 -0.0524849102 rpy=-0.543269873 -1.26599038 1.57079633
- added joint top_camera_right_optical_joint: type fixed, parent top_camera_camera, child top_camera_right_optical, origin xyz=0.424482885 -0.114380749 0.0619837129 rpy=-0.543269873 -1.26599038 1.57079633

File: src/linker_robot_assets/assets/workstations/ar5_l6_bench_bimanual/workstation.urdf (robot description, URDF)
Before this commit: robot ar5_l6_bench_bimanual, 58 links, 57 joints
Links:
- removed link base_camera
- removed link base_camera_base_link
- added link base_workstation_camera_mount
- added link top_camera_camera, mass 0.170230156191785; collision mesh filename=../../components/sensors/workstation_zed2i/variants/default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; visual mesh filename=../../components/sensors/workstation_zed2i/variants/default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
- added link top_camera_camera_base_link, mass 0.120253078965696; collision mesh filename=../../components/sensors/workstation_zed2i/variants/default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; visual mesh filename=../../components/sensors/workstation_zed2i/variants/default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
- added link top_camera_left_optical, mass 1e-9
- added link top_camera_right_optical, mass 1e-9
Joints:
- removed joint base_cameraBase
- removed joint base_cameraJoint
- added joint base_weld_workstation_camera_mount: type fixed, parent base_workstation_link, child base_workstation_camera_mount, origin xyz=0.0335 0.67 1.2974 rpy=-1.5708 0 -1.5708
- added joint mount_top_camera_to_base_base_mount: type fixed, parent base_workstation_camera_mount, child top_camera_camera_base_link, origin xyz=0 0 0 rpy=0 0 0
- added joint top_camera_cameraJoint: type fixed, parent top_camera_camera_base_link, child top_camera_camera, origin xyz=0.0802 0.193139854 -0.275851476 rpy=-1.26599038 -0.643554018 -1.57079633, axis 0 0 0
- added joint top_camera_left_optical_joint: type fixed, parent top_camera_camera, child top_camera_left_optical, origin xyz=0.424482885 -0.150393718 -0.0524849102 rpy=-0.543269873 -1.26599038 1.57079633
- added joint top_camera_right_optical_joint: type fixed, parent top_camera_camera, child top_camera_right_optical, origin xyz=0.424482885 -0.114380749 0.0619837129 rpy=-0.543269873 -1.26599038 1.57079633

File: src/linker_robot_assets/assets/workstations/ar5_o6_bench_bimanual/workstation.urdf (robot description, URDF)
Before this commit: robot ar5_o6_bench_bimanual, 48 links, 47 joints
Links:
- removed link base_camera
- removed link base_camera_base_link
- added link base_workstation_camera_mount
- added link top_camera_camera, mass 0.170230156191785; collision mesh filename=../../components/sensors/workstation_zed2i/variants/default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; visual mesh filename=../../components/sensors/workstation_zed2i/variants/default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
- added link top_camera_camera_base_link, mass 0.120253078965696; collision mesh filename=../../components/sensors/workstation_zed2i/variants/default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; visual mesh filename=../../components/sensors/workstation_zed2i/variants/default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
- added link top_camera_left_optical, mass 1e-9
- added link top_camera_right_optical, mass 1e-9
Joints:
- removed joint base_cameraBase
- removed joint base_cameraJoint
- added joint base_weld_workstation_camera_mount: type fixed, parent base_workstation_link, child base_workstation_camera_mount, origin xyz=0.0335 0.67 1.2974 rpy=-1.5708 0 -1.5708
- added joint mount_top_camera_to_base_base_mount: type fixed, parent base_workstation_camera_mount, child top_camera_camera_base_link, origin xyz=0 0 0 rpy=0 0 0
- added joint top_camera_cameraJoint: type fixed, parent top_camera_camera_base_link, child top_camera_camera, origin xyz=0.0802 0.193139854 -0.275851476 rpy=-1.26599038 -0.643554018 -1.57079633, axis 0 0 0
- added joint top_camera_left_optical_joint: type fixed, parent top_camera_camera, child top_camera_left_optical, origin xyz=0.424482885 -0.150393718 -0.0524849102 rpy=-0.543269873 -1.26599038 1.57079633
- added joint top_camera_right_optical_joint: type fixed, parent top_camera_camera, child top_camera_right_optical, origin xyz=0.424482885 -0.114380749 0.0619837129 rpy=-0.543269873 -1.26599038 1.57079633
